Commit message: Update crawler model

File: crawler_description/urdf/crawler.xacro (robot description, xacro)
@@ -17,4 +17,5 @@
   <xacro:property name="front_wheel_y_offset" value="0.070"/>
   <xacro:property name="front_wheel_z_offset" value="-0.03"/>
+  <xacro:property name="front_wheel_mass" value="0.5"/>
   <!-- Rear wheel is a caster wheel but we represent it with a
        sphere -->
@@ -26,19 +27,7 @@
   <xacro:property name="rear_wheel_y_offset" value="0.0"/>
   <xacro:property name="rear_wheel_z_offset" value="-0.035"/>
+  <xacro:property name="rear_wheel_mass" value="0.5"/>
   <!-- Plugin Variables-->
   <xacro:property name="wheel_separation" value="0.138"/>
-  <!--Color Properties-->
-  <material name="blue">
-    <color rgba="0 0 0.8 1"/>
-  </material>
-  <material name="black">
-    <color rgba="0 0 0 1"/>
-  </material>
-  <material name="white">
-    <color rgba="1 1 1 1"/>
-  </material>
-  <material name="red">
-    <color rgba="0.8 0.0 0.0 1.0"/>
-  </material>
   <!--Interial macros-->
   <xacro:macro name="cylinder_inertia" params="m r h">
@@ -69,10 +58,10 @@
     <origin xyz="0 0 0" rpy="0 0 0" />
     <xacro:box_inertia m="0.01" w="${base_len}" h="${base_width}" d="${base_depth}"/>
-    <visual>
+    <!-- <visual>
       <origin xyz="-0.03 0 0.03" rpy="-1.57 0 -1.57"/>
       <geometry>
         <mesh filename="file:///$(find crawler_description)/meshes/Altiscan2t_no_wheels.dae"/>
       </geometry>
-    </visual>
+    </visual> -->
     <collision>
       <geometry>
@@ -110,5 +99,5 @@
         </friction>
       </surface>
-      <xacro:cylinder_inertia m=".5" r="${front_wheel_radius}" h="${front_wheel_length}"/>
+      <xacro:cylinder_inertia m="${front_wheel_mass}" r="${front_wheel_radius}" h="${front_wheel_length}"/>
     </link>
     <joint name="${prefix}_front_wheel_joint" type="continuous">
@@ -138,5 +127,5 @@
     <parent link="caster_wheel_base"/>
     <child link="caster_wheel"/>
-    <origin xyz="${rear_wheel_arm} 0 ${rear_wheel_z_offset}" rpy="0 0 0"/>
+    <origin xyz="${-rear_wheel_arm} 0 ${rear_wheel_z_offset}" rpy="0 0 0"/>
   </joint>
   <link name="caster_wheel">
@@ -161,11 +150,5 @@
       </friction>
     </surface>
-    <xacro:cylinder_inertia m="0.5" r="${rear_wheel_radius}" h="${rear_wheel_width}"/>
+    <xacro:cylinder_inertia m="${rear_wheel_mass}" r="${rear_wheel_radius}" h="${rear_wheel_width}"/>
   </link>
-  <xacro:property name="imu_size_x" value="0.003"/>
-  <xacro:property name="imu_size_y" value="0.003"/>
-  <xacro:property name="imu_size_z" value="0.001"/>
-  <xacro:property name="imu_origin_x" value="-0.10"/>
-  <xacro:property name="imu_origin_y" value="-0.15"/>
-  <xacro:property name="imu_origin_z" value="0.00"/>
 </robot>

File: crawler_description/urdf/crawler_caster.urdf (robot description, URDF)
Before this commit: robot crawler, 6 links, 5 joints
Links:
- link base_link: mass 0.01 -> 2; geometry collision box size=0.2 0.2 0.05
- link caster_wheel: mass 0.25 -> 0.5; geometry collision cylinder length=0.04 radius=0.02; visual cylinder length=0.04 radius=0.02
- link caster_wheel_base: geometry visual box size=0.13 0.01 0.01
- link left_front_wheel: mass 0.5 -> 0.8
- link right_front_wheel: mass 0.5 -> 0.8
Joints:
- joint caster_wheel_joint: origin xyz=-0.088 0.0 -0.0325 rpy=0 0 0 -> xyz=-0.02 0 -0.035 rpy=0 0 0; parent base_link -> caster_wheel_base

File: crawler_description/urdf/crawler_sphere.urdf (robot description, URDF)
Before this commit: robot crawler, 5 links, 4 joints
Links:
- link base_link: mass 0.01 -> 2; geometry collision box size=0.2 0.2 0.05
- link left_front_wheel: mass 0.5 -> 0.8
- link right_front_wheel: mass 0.5 -> 0.8
